Commit message: Constrain workspace to front collision-free region

File: simulation/urdf/home_mobile_manipulator_v6_real_base_layout.urdf (robot description, URDF)
Before this commit: robot home_mobile_manipulator_v6_real_base_layout, 33 links, 32 joints
Links:
- link arm_base_mount: geometry collision box size=0.060 0.080 0.080; visual box size=0.060 0.080 0.080
- link elbow_servo: geometry collision box size=0.050 0.050 0.050; visual box size=0.050 0.050 0.050
- link forearm: geometry collision box size=0.110 0.045 0.045; visual box size=0.110 0.045 0.045
- link gripper: geometry collision box size=0.100 0.070 0.055; visual box size=0.100 0.070 0.055
- link shoulder_servo: geometry collision box size=0.050 0.050 0.050; visual box size=0.050 0.050 0.050
- link upper_arm: geometry collision box size=0.120 0.045 0.045; visual box size=0.120 0.045 0.045
- link wrist_roll_link: geometry collision box size=0.080 0.040 0.040; visual box size=0.080 0.040 0.040
- link wrist_servo: geometry collision box size=0.048 0.048 0.048; visual box size=0.048 0.048 0.048
